File: hardware/dmxfire16.kicad_pcb (KiCad board)
At the start: 2 copper layers, 203.2 x 82.5 mm, 159 parts, among them J1 IN, J2 OUT, P1 SOL1, P10 SOL10, P11 SOL11, P12 SOL12, P13 SOL13, P14 SOL14, P15 SOL15, P16 SOL16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

Commit message: removing named pin
Parts:
- JP3: value TERM -> TERMINATION
Connections:
- net /CLEAR renamed Net-(P23-Pad5)
Other:
- board text added: "4"
- board text removed: "CLEAR"

Commit message: slight silk change
Parts:
- JP3: value TERMINATION -> TERM
